File: pcb/Grinder.kicad_pcb (KiCad board)
At the start: 2 copper layers, 43.2 x 57.1 mm, 8 parts

Commit message: WIP for new PCB
Parts:
- removed IRF520N: TO-220-3_Vertical, Package_TO_SOT_THT:TO-220-3_Vertical
- removed the LED at (148.6, 59.7)
- removed R1 1K: R_Box_L8.4mm_W2.5mm_P5.08mm, Resistor_THT:R_Box_L8.4mm_W2.5mm_P5.08mm
- removed R2 1K: R_Box_L8.4mm_W2.5mm_P5.08mm, Resistor_THT:R_Box_L8.4mm_W2.5mm_P5.08mm
- added ADS1232: TSSOP-24_4.4x7.8mm_P0.65mm, Package_SO:TSSOP-24_4.4x7.8mm_P0.65mm, F.Cu at (159.0, 67.9)
- added C1: C_0201_0603Metric, Capacitor_SMD:C_0201_0603Metric, F.Cu at (157.0, 63.0)
- added LED: LED_0201_0603Metric, LED_SMD:LED_0201_0603Metric, F.Cu at (138.4, 75.9)
- added Load cell: PinSocket_1x04_P2.54mm_Vertical, Connector_PinSocket_2.54mm:PinSocket_1x04_P2.54mm_Vertical, F.Cu at (172.7, 58.4)
- added R1: R_0201_0603Metric, Resistor_SMD:R_0201_0603Metric, F.Cu at (140.7, 75.9)
- added R2: R_0201_0603Metric, Resistor_SMD:R_0201_0603Metric, F.Cu at (140.7, 77.5)
- added REF**: C_0201_0603Metric, Capacitor_SMD:C_0201_0603Metric, F.Cu at (158.8, 72.9)
- added REF**: R_0201_0603Metric, Resistor_SMD:R_0201_0603Metric, F.Cu at (168.4, 66.0)
- added REF**: R_0201_0603Metric, Resistor_SMD:R_0201_0603Metric, F.Cu at (168.4, 63.5)
- added REF**: R_0201_0603Metric, Resistor_SMD:R_0201_0603Metric, F.Cu at (154.7, 75.2)
- added REF**: R_0201_0603Metric, Resistor_SMD:R_0201_0603Metric, F.Cu at (154.7, 73.9)
- added REF**: C_0201_0603Metric, Capacitor_SMD:C_0201_0603Metric, F.Cu at (157.0, 72.9)
- added REF**: Battery_CR1225, Battery:Battery_CR1225, F.Cu at (142.0, 75.9)
- added REF**: TO-263-2, Package_TO_SOT_SMD:TO-263-2, F.Cu at (147.0, 64.1)
- added REF**: TO-252-2, Package_TO_SOT_SMD:TO-252-2, F.Cu at (135.0, 61.4)
- added REF**: C_0201_0603Metric, Capacitor_SMD:C_0201_0603Metric, F.Cu at (162.3, 63.0)
- added REF**: C_0201_0603Metric, Capacitor_SMD:C_0201_0603Metric, F.Cu at (166.6, 64.8)
- moved Rotary Enc. 15.5 mm to (135.9, 114.3)
- moved UEXT 15.3 mm to (154.9, 114.3)
- moved Arduino Nano 12.8 mm to (132.1, 100.3)
- moved REF** 2.54 mm to (138.4, 48.3)
- renumbered OLED to UEXT
Routing:
- net (no net): track 434.8 -> 972.4 mm, vias 0 -> 4
Other:
- board size 43.2 x 57.1 mm -> 48 x 73 mm
- net class 5V added: clearance 0.2, trace_width 0.25, via_dia 0.8, via_drill 0.4
- net class 9V added: clearance 0.2, trace_width 0.25, via_dia 0.8, via_drill 0.4
- board text added: "A+"
- board text added: "A-"
- board text added: "ADC CLK"
- board text added: "ADC DOUT"
- board text added: "ADC PDWN"
- board text added: "ADC SPD"
- board text added: "E+"
- board text added: "E-"
- board text added: "MISO"
- board text added: "MOSI"
- board text added: "RX"
- board text added: "RXD"
- board text added: "SCK"
- board text added: "SSEL"
- board text added: "TX"
- board text added: "TXD"
- board text removed: "D"
- board text removed: "G"
- board text removed: "S"

Commit message: WIP
Parts:
- removed ADS1232: TSSOP-24_4.4x7.8mm_P0.65mm, Package_SO:TSSOP-24_4.4x7.8mm_P0.65mm
- removed Arduino Nano: Arduino_Nano, Module:Arduino_Nano
- removed LED: LED_0201_0603Metric, LED_SMD:LED_0201_0603Metric
- removed the REF** at (158.8, 72.9)
- removed the REF** at (168.4, 66.0)
- removed the REF** at (168.4, 63.5)
- removed the REF** at (154.7, 75.2)
- removed the REF** at (154.7, 73.9)
- removed the REF** at (157.0, 72.9)
- removed the REF** at (142.0, 75.9)
- removed the REF** at (147.0, 64.1)
- removed the REF** at (135.0, 61.4)
- removed the REF** at (162.3, 63.0)
- removed the REF** at (166.6, 64.8)
- added A1: Arduino Nano 33 IoT, Module:Arduino_Nano, F.Cu at (132.1, 100.3)
- added C2: 10 nF, Capacitor_SMD:C_0402_1005Metric, F.Cu at (166.4, 65.1)
- added C3: 100 nF, Capacitor_SMD:C_0402_1005Metric, F.Cu at (155.7, 59.7)
- added C4: 100nF, Capacitor_SMD:C_0402_1005Metric, F.Cu at (163.9, 58.8)
- added D1: LED, LED_SMD:LED_0805_2012Metric, F.Cu at (134.6, 77.5)
- added Q1: IRLZ44N, Package_TO_SOT_SMD:TO-263-2, F.Cu at (138.2, 65.5)
- added R3: 100R, Resistor_SMD:R_0402_1005Metric, F.Cu at (156.5, 72.9)
- added R4: 100R, Resistor_SMD:R_0402_1005Metric, F.Cu at (154.9, 72.9)
- added R5: 100R, Resistor_SMD:R_0402_1005Metric, F.Cu at (168.4, 64.3)
- added R6: 100R, Resistor_SMD:R_0402_1005Metric, F.Cu at (168.4, 65.8)
- added REF**: MountingHole_2.2mm_M2, MountingHole:MountingHole_2.2mm_M2, F.Cu at (129.0, 109.5)
- added REF**: MountingHole_2.2mm_M2, MountingHole:MountingHole_2.2mm_M2, F.Cu at (173.0, 109.5)
- added REF**: MountingHole_2.2mm_M2, MountingHole:MountingHole_2.2mm_M2, F.Cu at (173.0, 52.5)
- added REF**: MountingHole_2.2mm_M2, MountingHole:MountingHole_2.2mm_M2, F.Cu at (129.0, 52.5)
- added U1: ADS1232IPW, Package_SO:TSSOP-24_4.4x7.8mm_P0.65mm, F.Cu at (157.7, 65.1)
- C1: value C_0201_0603Metric -> 10nF; footprint Capacitor_SMD:C_0201_0603Metric -> Capacitor_SMD:C_0402_1005Metric
- J1: renamed from REF**; value TerminalBlock_bornier-6_P5.08mm -> Conn_01x06
- J2: renamed from Rotary Enc.; value PinHeader_1x05_P2.54mm_Vertical -> Conn_01x05
- J3: renamed from Load cell; value PinSocket_1x04_P2.54mm_Vertical -> Conn_01x04
- J4: renamed from UEXT; value PinHeader_2x05_P2.54mm_Vertical -> Conn_02x05_Odd_Even
- R1, R2: value R_0201_0603Metric -> R; footprint Resistor_SMD:R_0201_0603Metric -> Resistor_SMD:R_0402_1005Metric
- moved C1 8.23 mm to (155.7, 71.1)
- moved R1 3.21 mm to (137.7, 77.0)
- moved R2 3.14 mm to (137.7, 78.2)
Connections:
- C1 pad 1: (no net) -> GNDA
- C1 pad 2: (no net) -> 5V_FILTERED
- J1 pad 1: (no net) -> 5V
- J1 pad 2: (no net) -> GND
- J1 pad 3: (no net) -> 5V
- J1 pad 4: (no net) -> SSR_DRAIN
- J1 pad 5: (no net) -> MANUAL_SW
- J1 pad 6: (no net) -> GND
- J2 pad 1: (no net) -> ENC_CLK
- J2 pad 2: (no net) -> ENC_DT
- J2 pad 3: (no net) -> ENC_SW
- J2 pad 4: (no net) -> 3V3
- J2 pad 5: (no net) -> GND
- J3 pad 1: (no net) -> 5V
- J3 pad 2: (no net) -> GND
- J3 pad 3: (no net) -> Net-(J3-Pad3)
- J3 pad 4: (no net) -> Net-(J3-Pad4)
- J4 pad 1: (no net) -> 3V3
- J4 pad 10: (no net) -> UEXT_SSEL
- J4 pad 2: (no net) -> GND
- J4 pad 3: (no net) -> UEXT_TX
- J4 pad 4: (no net) -> UEXT_RX
- J4 pad 5: (no net) -> UEXT_SCL
- J4 pad 6: (no net) -> UEXT_SDA
- J4 pad 7: (no net) -> UEXT_MISO
- J4 pad 8: (no net) -> UEXT_MOSI
- J4 pad 9: (no net) -> UEXT_SCK
- R1 pad 1: (no net) -> Net-(D1-Pad2)
- R1 pad 2: (no net) -> SSR_GATE
- R2 pad 1: (no net) -> GND
- R2 pad 2: (no net) -> SSR_GATE
Routing:
- net (no net): track 972.4 -> 0.00 mm, vias 4 -> 0
- net GND: track 0.00 -> 219.3 mm
- net 5V: track 0.00 -> 145.6 mm, vias 0 -> 2
- net 3V3: track 0.00 -> 75.8 mm
- net MANUAL_SW: track 0.00 -> 37.4 mm
- net UEXT_TX: track 0.00 -> 36.7 mm
- net UEXT_SCL: track 0.00 -> 34.5 mm
- net UEXT_RX: track 0.00 -> 32.5 mm
- net UEXT_SCK: track 0.00 -> 31.6 mm
- net UEXT_SDA: track 0.00 -> 30.9 mm
- net Net-(C2-Pad2): track 0.00 -> 28.6 mm, vias 0 -> 2
- net ADC_SPEED: track 0.00 -> 27.1 mm
- net Net-(C2-Pad1): track 0.00 -> 24.3 mm, vias 0 -> 2
- net SSR_DRAIN: track 0.00 -> 23.8 mm
- net UEXT_SSEL: track 0.00 -> 20.4 mm
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Other:
- net class 9V removed
- board text added: "FB 20"

Commit message: WIP
Parts:
- removed C3: 100 nF, Capacitor_SMD:C_0402_1005Metric
- removed C4: 100nF, Capacitor_SMD:C_0402_1005Metric
- Q1: footprint Package_TO_SOT_SMD:TO-263-2 -> Package_TO_SOT_THT:TO-220-3_Horizontal_TabDown
- U1: value ADS1232IPW -> CJMCU-ADS1232; footprint Package_SO:TSSOP-24_4.4x7.8mm_P0.65mm -> custom:DIP-18_600
- moved R4 19.4 mm to (163.8, 55.6), turned to 270 degrees
- moved R3 19.3 mm to (165.1, 55.6), turned to 270 degrees
- moved C1 16.2 mm to (164.3, 57.4)
- moved Q1 10.3 mm to (136.7, 75.7), turned to 0 degrees
- moved C2 10.2 mm to (172.2, 73.4), turned to 0 degrees
- moved R5 7.50 mm to (171.4, 71.1), turned to 90 degrees
- moved R6 7.19 mm to (173.2, 71.1), turned to 90 degrees
- moved D1 5.92 mm to (139.7, 80.5), turned to 180 degrees
- moved U1 5.55 mm to (157.5, 70.6)
- moved R1 3.14 mm to (136.9, 80.0)
- moved R2 3.14 mm to (136.9, 81.3)
Connections:
- C2 pad 1: Net-(C2-Pad1) -> ADC_AINP1
- C2 pad 2: Net-(C2-Pad2) -> ADC_AINN1
- D1 pad 1: GND -> Net-(D1-Pad1)
- D1 pad 2: Net-(D1-Pad2) -> SSR_GATE
- J3 pad 1: 5V -> 5V_FILTERED
- R1 pad 1: Net-(D1-Pad2) -> GND
- R1 pad 2: SSR_GATE -> Net-(D1-Pad1)
- R5 pad 1: Net-(C2-Pad1) -> ADC_AINP1
- R6 pad 1: Net-(C2-Pad2) -> ADC_AINN1
- U1 pad 10: Net-(C3-Pad2) -> 3V3
- U1 pad 11: Net-(C2-Pad1) -> GNDA
- U1 pad 12: Net-(C2-Pad2) -> GNDA
- U1 pad 13: Net-(U1-Pad13) -> GNDA
- U1 pad 14: Net-(U1-Pad14) -> GNDA
- U1 pad 15: GNDA -> ADC_AINN1
- U1 pad 16: 5V_FILTERED -> ADC_AINP1
- U1 pad 17: GND -> Net-(U1-Pad17)
- U1 pad 18: 5V -> Net-(U1-Pad18)
- U1 pad 2: GND -> 3V3
- U1 pad 3: GND -> ADC_SPEED
- U1 pad 4: Net-(U1-Pad4) -> ADC_PDWN
- U1 pad 5: GND -> ADC_DOUT
- U1 pad 6: GND -> ADC_CLK
- U1 pad 7: GND -> 5V_FILTERED
- U1 pad 8: GND -> GNDA
- U1 pad 9: Net-(C3-Pad1) -> 5V_FILTERED
Routing:
- net GND: track 219.3 -> 133.6 mm
- net 5V: track 145.6 -> 80.2 mm, vias 2 -> 0
- net 5V_FILTERED: track 4.63 -> 52.2 mm
- net GNDA: track 4.66 -> 37.6 mm
- net Net-(C2-Pad2): track 28.6 -> 0.00 mm, vias 2 -> 0
- net Net-(C2-Pad1): track 24.3 -> 0.00 mm, vias 2 -> 0
- net ADC_AINP1: track 0.00 -> 18.1 mm
- net ADC_AINN1: track 0.00 -> 15.1 mm
- net SSR_DRAIN: track 23.8 -> 33.4 mm
- net ADC_CLK: track 19.5 -> 14.0 mm
- net ADC_SPEED: track 27.1 -> 22.7 mm
- net Net-(D1-Pad1): track 0.00 -> 3.86 mm
- net Net-(J3-Pad3): track 4.12 -> 7.64 mm
- net SSR_GATE: track 16.5 -> 19.4 mm
- net MANUAL_SW: track 37.4 -> 40.0 mm, vias 0 -> 1
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